File: KillSwitch_pcb/KillSwitchIO.kicad_sch (KiCad schematic)
At the start: 30 parts, among them SW5 KILL1, SW6 KILL2, SW7 KILL3, SW8 KILL4, U2 MCP23017_SO

Commit message: replace 100nF caps with 470nf
Parts:
- C10: value 100nF -> 470nF
Changed lines of the file:
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@@
 			)
 		)
-		(property "Value" "100nF"
+		(property "Value" "470nF"
 			(at 48.768 47.498 0)
 			(effects
